File: hardware/orangecrab_r0.1/bosonFrameGrabber.sch (KiCad schematic (older format))
At the start: 0 parts

Commit message: Update schematic
Changed lines of the file:
@@
 $Descr A4 11693 8268
 encoding utf-8
-Sheet 1 5
+Sheet 1 6
 Title ""
 Date ""
@@
 F1 "fileIO.sch" 60
 $EndSheet
+$Sheet
+S 1800 2900 1900 900
+U 5D1738DB
+F0 "sheetPower" 60
+F1 "filePOWER.sch" 60
+$EndSheet
 $EndSCHEMATC
