File: hardware/orangecrab_r0.1/fileSDMMC.sch (KiCad schematic (older format))
At the start: 6 parts, among them J4 MicroSd

Commit message: Update PN/MFG of resistor packs
Parts:
- RN7: Mfg Vishay Dale -> Stackpole Electronics Inc; PN CRA06S08310K0JTA -> RAVF104DJT10K0
Changed lines of the file:
@@
 F 2 "Resistor_SMD:R_Array_Convex_4x0402" V 3125 2950 50  0001 C CNN
 F 3 "~" H 2850 2950 50  0001 C CNN
-F 4 "CRA06S08310K0JTA" H 2850 2950 50  0001 C CNN "PN"
-F 5 "Vishay Dale" H 2850 2950 50  0001 C CNN "Mfg"
+F 4 "RAVF104DJT10K0" H 2850 2950 50  0001 C CNN "PN"
+F 5 "Stackpole Electronics Inc" H 2850 2950 50  0001 C CNN "Mfg"
 	1    2850 2950
 	1    0    0    -1
