File: hardware/orangecrab_r0.2/filePOWER.sch (KiCad schematic (older format))
At the start: 48 parts, among them J5 JST, U1 FAN53541, U10 NCP115-2.5, U2 FAN53541, U5 BQ24232, U7 FAN53541, U8 TPS51206

Commit message: hw: Update I/O block routing new DDR3 signals.
Parts:
- U10: footprint gkl_housings_son:X2SON_4_1.0x1.0mm -> Package_SON:Texas_X2SON-4_1x1mm_P0.65mm
Changed lines of the file:
@@
 F 0 "U10" H 3350 4968 50  0000 C CNN
 F 1 "NCP115-2.5" H 3350 4877 50  0000 C CNN
-F 2 "gkl_housings_son:X2SON_4_1.0x1.0mm" H 3300 4950 50  0001 C CNN
+F 2 "Package_SON:Texas_X2SON-4_1x1mm_P0.65mm" H 3300 4950 50  0001 C CNN
 F 3 "" H 3350 4850 50  0001 C CNN
 F 4 "NCP115CMX250TCG" H 3350 4600 50  0001 C CNN "PN"

Commit message: hw: Update board with 3d models Finish pin-swaps and routing of open changes General cleanups
Parts:
- removed R6: 0R, Resistor_SMD:R_0402_1005Metric, symbol Device:R
Connections:
- net P1.35V: now also C8.2, U8.2 (VLDOIN)
Changed lines of the file:
@@
 Text GLabel 1450 5950 0    50   UnSpc ~ 0
 P1.35V
-Wire Wire Line
-	1550 5950 1450 5950
-$Comp
-L Device:R R?
-U 1 1 5D20B7E1
-P 1700 5950
-AR Path="/5ABD38F2/5D20B7E1" Ref="R?"  Part="1"
-AR Path="/5D1738DB/5D20B7E1" Ref="R6"  Part="1"
-F 0 "R6" V 1493 5950 50  0000 C CNN
-F 1 "0R" V 1584 5950 50  0000 C CNN
-F 2 "Resistor_SMD:R_0402_1005Metric" V 1630 5950 50  0001 C CNN
-F 3 "~" H 1700 5950 50  0001 C CNN
-F 4 "‎Yageo‎" H 1700 5950 50  0001 C CNN "Mfg"
-F 5 "RC0402FR-070RL" H 1700 5950 50  0001 C CNN "PN"
-	1    1700 5950
-	0    1    1    0
-$EndComp
 Connection ~ 2000 5950
-Wire Wire Line
-	2000 5950 1850 5950
 Wire Wire Line
 	2000 5950 2800 5950
@@
 Text Notes 9600 6100 0    50   ~ 0
 3.3V
+Wire Wire Line
+	1450 5950 2000 5950
 $EndSCHEMATC

Commit message: hardware/orangecrab_r0.2: r0.2 Release
Prepared KiCad files for release
Create production folder
Add pdf schematic
Parts:
- R16: PN RC0201FR-07115KL -> RC0201FR-07147KL
- R26: value 10K -> 10k
- R7: value 1.5K -> 10k; PN RC0201FR-071K5L -> RC0201FR-0710KL
- R8: value 1.5K -> 4.7k; PN RC0201FR-071K5L -> RC0201FR-074K7L
Changed lines of the file:
@@
 EESchema Schematic File Version 4
-LIBS:OrangeCrab-cache
 EELAYER 30 0
 EELAYER END
@@
 Sheet 6 7
 Title "Orange Crab"
-Date "2019-06-28"
-Rev "r0.1"
-Comp "GsD"
+Date "2019-12-08"
+Rev "r0.2"
+Comp "Good Stuff Department"
 Comment1 ""
 Comment2 ""
-Comment3 ""
-Comment4 ""
+Comment3 "Licensed under CERN OHL v.1.2"
+Comment4 "Designed by: Greg Davill"
 $EndDescr
 Text Notes 6100 2050 2    50   ~ 0
@@
 F 3 "~" H 9450 4050 50  0001 C CNN
 F 4 "‎Yageo‎" H 9450 4050 50  0001 C CNN "Mfg"
-F 5 "RC0201FR-07115KL" H 9450 4050 50  0001 C CNN "PN"
+F 5 "RC0201FR-07147KL" H 9450 4050 50  0001 C CNN "PN"
 	1    9450 4050
 	1    0    0    -1
@@
 P 1450 3500
 F 0 "R8" V 1565 3500 50  0000 C CNN
-F 1 "1.5K" V 1656 3500 50  0000 C CNN
+F 1 "4.7k" V 1656 3500 50  0000 C CNN
 F 2 "Resistor_SMD:R_0201_0603Metric" V 1380 3500 50  0001 C CNN
 F 3 "~" H 1450 3500 50  0001 C CNN
 F 4 "‎Yageo‎" H 1450 3500 50  0001 C CNN "Mfg"
-F 5 "RC0201FR-071K5L" H 1450 3500 50  0001 C CNN "PN"
+F 5 "RC0201FR-074K7L" H 1450 3500 50  0001 C CNN "PN"
 	1    1450 3500
 	0    1    1    0
@@
 P 1450 3300
 F 0 "R7" V 1243 3300 50  0000 C CNN
-F 1 "1.5K" V 1334 3300 50  0000 C CNN
+F 1 "10k" V 1334 3300 50  0000 C CNN
 F 2 "Resistor_SMD:R_0201_0603Metric" V 1380 3300 50  0001 C CNN
 F 3 "~" H 1450 3300 50  0001 C CNN
 F 4 "‎Yageo‎" H 1450 3300 50  0001 C CNN "Mfg"
-F 5 "RC0201FR-071K5L" H 1450 3300 50  0001 C CNN "PN"
+F 5 "RC0201FR-0710KL" H 1450 3300 50  0001 C CNN "PN"
 	1    1450 3300
 	0    1    1    0
@@
 P 4250 2850
 F 0 "R26" H 4181 2804 50  0000 R CNN
-F 1 "10K" H 4181 2895 50  0000 R CNN
+F 1 "10k" H 4181 2895 50  0000 R CNN
 F 2 "Resistor_SMD:R_0201_0603Metric" V 4180 2850 50  0001 C CNN
 F 3 "~" H 4250 2850 50  0001 C CNN
